Commit message: ADD：修改了手眼相机的坐标系，添加了草莓的仿真模型

File: src/lerobot_description/urdf/so101.urdf.xacro (robot description, xacro)
@@ -4,3 +4,9 @@
     <xacro:include filename="$(find lerobot_description)/urdf/so101_gazebo.xacro" />
     <xacro:include filename="$(find lerobot_description)/urdf/so101_ros2_control.xacro" />
+    <xacro:include filename="$(find lerobot_description)/urdf/so101_camera_in_hand.xacro" />
+    <xacro:so101_camera_in_hand
+        parent="gripper"
+        origin_xyz="0.03 0.0 0.0"
+        origin_rpy="0 0 0"
+    />
 </robot>

File: src/lerobot_description/urdf/so101_base.xacro (robot description, xacro)
@@ -6,10 +6,10 @@
 -->
 <robot xmlns:xacro="http://www.ros.org/wiki/xacro">
-	<!-- Links -->
+    <!-- Links -->
 	<link name="world" />
 	<joint name="base_joint" type="fixed">
 		<parent link="world" />
 		<child link="base" />
-		<origin xyz="0 0 0" rpy="0 0 0" />
+		<origin xyz="0 0 0.175" rpy="0 0 0" />
 	</joint>
 	<!-- Materials -->
